Commit message: -

File: dualarm_mobile_description/urdf/base.gazebo.xacro (robot description, xacro)
@@ -4,21 +4,4 @@
        xmlns:interface="http://playerstage.sourceforge.net/gazebo/xmlschema/#interface"
        xmlns:xacro="http://ros.org/wiki/xacro">
-    <gazebo>
-        <plugin name="dummy_drive" filename="libgazebo_ros_planar_move.so">
-            <legacyMode>false</legacyMode>
-            <alwaysOn>true</alwaysOn>
-            <updateRate>100</updateRate>
-            <covariance_x>0.000100</covariance_x>
-            <covariance_y>0.000100</covariance_y>
-            <covariance_yaw>0.010000</covariance_yaw>
-            <broadcastTF>100</broadcastTF>
-            <torque>5</torque>
-            <commandTopic>cmd_vel</commandTopic>
-            <odometryTopic>odom</odometryTopic>
-            <odometryFrame>odom</odometryFrame>
-            <odometryRate>100.0</odometryRate>
-            <robotBaseFrame>base_footprint</robotBaseFrame>
-        </plugin>
-    </gazebo>
     <gazebo reference="base_link">
         <material>Gazebo/DarkGrey</material>
@@ -49,4 +32,16 @@
         <material>Gazebo/FlatBlack</material>
     </gazebo>
+    <!-- <gazebo>
+      <plugin name="p3d_base_controller" filename="libgazebo_ros_p3d.so">
+        <alwaysOn>true</alwaysOn>
+        <updateRate>50.0</updateRate>
+        <bodyName>base_footprint</bodyName>
+        <topicName>pose</topicName>
+        <gaussianNoise>0.01</gaussianNoise>
+        <frameName>world</frameName>
+        <xyzOffsets>0 0 0</xyzOffsets>
+        <rpyOffsets>0 0 0</rpyOffsets>
+      </plugin>
+    </gazebo> -->
     <gazebo>
         <plugin name="imu_plugin" filename="libgazebo_ros_imu.so">
@@ -258,6 +253,6 @@
             <horizontal_fov>1.3962634</horizontal_fov>
             <image>
-            <width>720</width>
-            <height>480</height>
+            <width>128</width>
+            <height>96</height>
             <format>R8G8B8</format>
             </image>
@@ -295,6 +290,6 @@
             <horizontal_fov>1.3962634</horizontal_fov>
             <image>
-            <width>720</width>
-            <height>480</height>
+            <width>128</width>
+            <height>96</height>
             <format>R8G8B8</format>
             </image>
@@ -326,3 +321,20 @@
         </sensor>
     </gazebo>
+    <gazebo>
+        <plugin name="dummy_drive" filename="libgazebo_ros_planar_move.so">
+            <legacyMode>false</legacyMode>
+            <alwaysOn>true</alwaysOn>
+            <updateRate>100</updateRate>
+            <covariance_x>0.000100</covariance_x>
+            <covariance_y>0.000100</covariance_y>
+            <covariance_yaw>0.010000</covariance_yaw>
+            <broadcastTF>100</broadcastTF>
+            <torque>5</torque>
+            <commandTopic>cmd_vel</commandTopic>
+            <odometryTopic>odom</odometryTopic>
+            <odometryFrame>odom</odometryFrame>
+            <odometryRate>100.0</odometryRate>
+            <robotBaseFrame>base_footprint</robotBaseFrame>
+        </plugin>
+    </gazebo>
 </robot>

File: dualarm_mobile_description/urdf/base.urdf.xacro (robot description, xacro)
@@ -8,5 +8,34 @@
     <xacro:include filename="$(find description_dual)/urdf/materials.urdf.xacro"/>
     <!-- Base footprint -->
-    <link name="base_footprint"/>
+    <link name="base_footprint">
+        <visual>
+            <origin xyz="0 0 0" rpy="0 0 0" />
+            <geometry>
+                <box size="0.001 0.001 0.001"/>
+            </geometry>
+            <material name="material_red"/>
+        </visual>
+    </link>
+    <!-- Base link -->
+    <link name="base_link">
+        <inertial>
+            <origin xyz="0 0 0" rpy="0 0 0" />
+            <mass value="13.2312244818196" />
+            <inertia ixx="0.967053548924663" ixy="0" ixz="0" iyy="1.30612724440363" iyz="0" izz="0.962964405480844" />
+        </inertial>
+        <visual>
+            <origin xyz="0 0 0" rpy="0 0 0" />
+            <geometry>
+                <mesh filename="package://description_dual/meshes/base_link.STL" />
+            </geometry>
+            <material name="material_light_grey"/>
+        </visual>
+        <collision>
+        <origin xyz="0 0 0" rpy="0 0 0" />
+            <geometry>
+                <mesh filename="package://description_dual/meshes/base_link.STL" />
+            </geometry>
+        </collision>
+    </link>
     <joint name="base_joint" type="fixed">
         <parent link="base_footprint"/>
@@ -14,25 +43,4 @@
         <origin xyz="0.0 0.0 0.0" rpy="0 0 0"/>
     </joint>
-    <!-- Base link -->
-    <link name="base_link">
-        <inertial>
-            <origin xyz="0 0 0" rpy="0 0 0" />
-            <mass value="13.2312244818196" />
-            <inertia ixx="0.967053548924663" ixy="0" ixz="0" iyy="1.30612724440363" iyz="0" izz="0.962964405480844" />
-        </inertial>
-        <visual>
-            <origin xyz="0 0 0" rpy="0 0 0" />
-            <geometry>
-                <mesh filename="package://description_dual/meshes/base_link.STL" />
-            </geometry>
-            <material name="material_light_grey"/>
-        </visual>
-        <collision>
-        <origin xyz="0 0 0" rpy="0 0 0" />
-            <geometry>
-                <mesh filename="package://description_dual/meshes/base_link.STL" />
-            </geometry>
-        </collision>
-    </link>
     <!-- Back right wheel -->
     <link name="br_wheel_link">
