Commit message: Add files via upload

File: dualarm_mobile_description/urdf/real_robot.urdf.xacro (robot description, xacro)
@@ -1,398 +1,380 @@
-<robot name="vehicle_v2" >
-<!-- Materials -->
-<material name="white">
-    <color rgba="1 1 1 1"/>
-</material>
-<material name="grey">
-    <color rgba="0.5 0.5 0.5 1"/>
-</material>
-<material name="light_grey">
-    <color rgba="0.6 0.6 0.6 1"/>
-</material>
-<material name="dark_grey">
-    <color rgba="0.3 0.3 0.3 1"/>
-</material>
-<material name="black">
-    <color rgba="0.1 0.1 0.1 1"/>
-</material>
-<material name="red">
-    <color rgba="1 0 0 1"/>
-</material>
-<material name="green">
-    <color rgba="0.0 0.8 0.0 1"/>
-</material>
-<material name="blue">
-    <color rgba="0.0 0.0 1.0 1"/>
-</material>
-<material name="grey_blue">
-    <color rgba="0.4 0.4 1.0 1"/>
-</material>
-<material name="orange">
-    <color rgba="1.0 0.7 0.0 1"/>
-</material>
-<!-- Base footprint -->
-<link name="base_footprint">
-    <inertial>
+<?xml version="1.0" ?>
+<robot name="vehicle_v2" xmlns:xacro="http://ros.org/wiki/xacro">
+    <!-- Materials -->
+    <material name="white">
+        <color rgba="1 1 1 1"/>
+    </material>
+    <material name="grey">
+        <color rgba="0.5 0.5 0.5 1"/>
+    </material>
+    <material name="light_grey">
+        <color rgba="0.6 0.6 0.6 1"/>
+    </material>
+    <material name="dark_grey">
+        <color rgba="0.3 0.3 0.3 1"/>
+    </material>
+    <material name="black">
+        <color rgba="0.1 0.1 0.1 1"/>
+    </material>
+    <material name="red">
+        <color rgba="1 0 0 1"/>
+    </material>
+    <material name="green">
+        <color rgba="0.0 0.8 0.0 1"/>
+    </material>
+    <material name="blue">
+        <color rgba="0.0 0.0 1.0 1"/>
+    </material>
+    <material name="grey_blue">
+        <color rgba="0.4 0.4 1.0 1"/>
+    </material>
+    <material name="orange">
+        <color rgba="1.0 0.7 0.0 1"/>
+    </material>
+    <!-- Base footprint -->
+    <link name="base_footprint"/>
+    <!-- Base link -->
+    <link name="base_link">
+        <inertial>
+            <origin xyz="0 0 0" rpy="0 0 0" />
+            <mass value="13.2312244818196" />
+            <inertia ixx="0.967053548924663" ixy="0" ixz="0" iyy="1.30612724440363" iyz="0" izz="0.962964405480844" />
+        </inertial>
+        <visual>
+            <origin xyz="0 0 0" rpy="0 0 0" />
+            <geometry>
+                <mesh filename="package://description_dual/meshes/base_link.STL" />
+            </geometry>
+            <material name="light_grey"/>
+        </visual>
+        <collision>
         <origin xyz="0 0 0" rpy="0 0 0" />
-        <mass value="0.1" />
-        <inertia ixx="1.0" ixy="0.0" ixz="0.0" iyy="1.0" iyz="0.0" izz="0.0" />
-    </inertial>
-    <visual>
-        <origin xyz="0 0 0" rpy="0 0 0" />
-        <geometry>
-            <box size="0.001 0.001 0.001"/>
-        </geometry>
-        <material name="red"/>
-    </visual>
-    <collision>
-    <origin xyz="0 0 0" rpy="0 0 0" />
-        <geometry>
-            <box size="0.001 0.001 0.001"/>
-        </geometry>
-    </collision>
-</link>
-<!-- Base link -->
-<link name="base_link">
-    <inertial>
-        <origin xyz="0 0 0" rpy="0 0 0" />
-        <mass value="13.2312244818196" />
-        <inertia ixx="0.967053548924663" ixy="0" ixz="0" iyy="1.30612724440363" iyz="0" izz="0.962964405480844" />
-    </inertial>
-    <visual>
-        <origin xyz="0 0 0" rpy="0 0 0" />
-        <geometry>
-            <mesh filename="package://description_dual/meshes/base_link.STL" />
-        </geometry>
-        <material name="light_grey"/>
-    </visual>
-    <collision>
-    <origin xyz="0 0 0" rpy="0 0 0" />
-        <geometry>
-            <mesh filename="package://description_dual/meshes/base_link.STL" />
-        </geometry>
-    </collision>
-</link>
-<joint name="base_joint" type="fixed">
-    <parent link="base_footprint"/>
-    <child link="base_link"/>
-    <origin xyz="0.0 0.0 0.0" rpy="0 0 0"/>
-</joint>
-<!-- Back right wheel -->
-<link name="br_wheel_link">
-    <inertial>
-        <origin xyz="0 0 0" rpy="0 0 0" />
-        <mass value="0.571565980810561" />
-        <inertia ixx="1" ixy="0" ixz="0" iyy="1" iyz="0" izz="1" />
-    </inertial>
-    <visual>
-        <origin xyz="0 0 0" rpy="0 0 0" />
-        <geometry>
-            <mesh filename="package://description_dual/meshes/br_wheel_link.STL" />
-        </geometry>
-        <material name="orange"/>
-    </visual>
-    <collision>
-        <origin xyz="0 0 0" rpy="0 1.5707 1.5707" />
-        <geometry>
-        <cylinder radius="0.076" length="0.079"/>
-        </geometry>
-    </collision>
-</link>
-<joint name="br_wheel_joint" type="continuous">
-    <origin xyz="-0.281 -0.215 -0.020" rpy="0 0 0" />
-    <parent link="base_link" />
-    <child link="br_wheel_link" />
-    <axis xyz="0 -1 0" />
-</joint>
-<!-- Back left wheel -->
-<link name="bl_wheel_link">
-    <inertial>
-        <origin xyz="0 0 0" rpy="0 0 0" />
-        <mass value="0.571565974939204" />
-        <inertia ixx="1" ixy="0" ixz="0" iyy="1" iyz="0" izz="1" />
-    </inertial>
-    <visual>
-        <origin xyz="0 0 0" rpy="0 0 0" />
-        <geometry>
-            <mesh filename="package://description_dual/meshes/bl_wheel_link.STL" />
-        </geometry>
-        <material name="orange"/>
-    </visual>
-    <collision>
-        <origin xyz="0 0 0" rpy="0 1.5707 1.5707" />
-        <geometry>
-        <cylinder radius="0.076" length="0.079"/>
-        </geometry>
-    </collision>
-</link>
-<joint name="bl_wheel_joint" type="continuous">
-    <origin xyz="-0.281 0.215 -0.020" rpy="0 0 0" />
-    <parent link="base_link" />
-    <child link="bl_wheel_link" />
-    <axis xyz="0 -1 0" />
-</joint>
-<!-- Front right wheel -->
-<link name="fr_wheel_link">
-    <inertial>
-        <origin xyz="0 0 0" rpy="0 0 0" />
-        <mass value="0.571565974847631" />
-        <inertia ixx="1" ixy="0" ixz="0" iyy="1" iyz="0" izz="1" />
-    </inertial>
-    <visual>
-        <origin xyz="0 0 0" rpy="0 0 0" />
-        <geometry>
-            <mesh filename="package://description_dual/meshes/fr_wheel_link.STL" />
-        </geometry>
-        <material name="orange"/>
-    </visual>
-    <collision>
-        <origin xyz="0 0 0" rpy="0 1.5707 1.5707" />
-        <geometry>
-        <cylinder radius="0.076" length="0.079"/>
-        </geometry>
-    </collision>
-</link>
-<joint name="fr_wheel_joint" type="continuous">
-    <origin xyz="0.281 -0.215 -0.020" rpy="0 0 0" />
-    <parent link="base_link" />
-    <child link="fr_wheel_link" />
-    <axis xyz="0 -1 0" />
-</joint>
-<!-- Front left wheel -->
-<link name="fl_wheel_link">
-    <inertial>
-        <origin xyz="0 0 0" rpy="0 0 0" />
-        <mass value="0.571565975000551" />
-        <inertia ixx="1" ixy="0" ixz="0" iyy="1" iyz="0" izz="1" />
-    </inertial>
-    <visual>
-        <origin xyz="0 0 0" rpy="0 0 0" />
-        <geometry>
-            <mesh filename="package://description_dual/meshes/fl_wheel_link.STL" />
-        </geometry>
-        <material name="orange"/>
-    </visual>
-    <collision>
-        <origin xyz="0 0 0" rpy="0 1.5707 1.5707" />
-        <geometry>
-        <cylinder radius="0.076" length="0.079"/>
-        </geometry>
-    </collision>
-</link>
-<joint name="fl_wheel_joint" type="continuous">
-    <origin xyz="0.281 0.215 -0.020" rpy="0 0 0" />
-    <parent link="base_link" />
-    <child link="fl_wheel_link" />
-    <axis xyz="0 -1 0" />
-</joint>
-<!-- IMU sensor -->
-<link name="imu_link"/>
-<joint name="imu_joint" type="fixed">
-    <parent link="base_link"/>
-    <child link="imu_link"/>
-    <origin xyz="0 0 0" rpy="0 0 0"/>
-</joint>
-<!-- Scan sensor -->
-<link name="base_scan">
-    <inertial>
-        <mass value="0.16"/>
-        <origin xyz="0 0 0.0"/>
-        <inertia ixx="0.1" ixy="0.0" ixz="0.0" iyy="0.1" iyz="0.0" izz="0.1"/>
-    </inertial>
-    <visual>
-        <origin xyz="0 0 0.0" rpy="0 0 0"/>
-        <geometry>
-            <mesh filename="package://description_dual/meshes/hokuyo.dae" />
-        </geometry>
-        <material name="dark_grey"/>
-    </visual>
-    <collision>
-        <origin xyz="0 0 0.0" rpy="0 0 0"/>
-        <geometry>
-            <mesh filename="package://description_dual/meshes/hokuyo_convex.dae" />
-        </geometry>
-    </collision>
-</link>
-<joint name="scan_joint" type="fixed">
-    <parent link="base_link"/>
-    <child link="base_scan"/>
-    <origin xyz="0 0 0.57" rpy="0 0 0"/>
-</joint>
-<!-- Front sonar sensor -->
-<link name="base_sonar_front">
-    <inertial>
-        <mass value="0.001" />
-        <origin xyz="0 0 0" rpy="0 0 0" />
-        <inertia ixx="0.000000017" ixy="0.0" ixz="0.0" iyy="0.000000017" iyz="0.0" izz="0.000000017"/>
-    </inertial>
-    <visual>
-        <origin xyz="0 0 0" rpy="0 0 0" />
-        <geometry>
-            <mesh filename="package://description_dual/meshes/max_sonar_ez4.dae"/>
-        </geometry>
-    </visual>
-    <collision>
-        <origin xyz="0 0 0" rpy="0 0 0" />
-        <geometry>
-            <box size="0.01 0.01 0.01" />
-        </geometry>
-    </collision>
-</link>
-<joint name="sonar_front_sensor_joint" type="fixed">
-    <parent link="base_link"/>
-    <child link="base_sonar_front"/>
-    <origin xyz="0.42 0 0.09" rpy="0 0 0"/>
-</joint>
-<!-- Rear sonar sensor -->
-<link name="base_sonar_rear">
-    <inertial>
-        <mass value="0.001" />
-        <origin xyz="0 0 0" rpy="0 0 0" />
-        <inertia ixx="0.000000017" ixy="0.0" ixz="0.0" iyy="0.000000017" iyz="0.0" izz="0.000000017"/>
-    </inertial>
-    <visual>
-        <origin xyz="0 0 0" rpy="0 0 0" />
-        <geometry>
-            <mesh filename="package://description_dual/meshes/max_sonar_ez4.dae"/>
-        </geometry>
-    </visual>
-    <collision>
-        <origin xyz="0 0 0" rpy="0 0 0" />
-        <geometry>
-            <box size="0.01 0.01 0.01" />
-        </geometry>
-    </collision>
-</link>
-<joint name="sonar_rear_sensor_joint" type="fixed">
-    <parent link="base_link"/>
-    <child link="base_sonar_rear"/>
-    <origin xyz="-0.41 0 0.09" rpy="0 0 3.1415926535897931"/>
-</joint>
-<!-- Left sonar sensor -->
-<link name="base_sonar_left">
-    <inertial>
-        <mass value="0.001" />
-        <origin xyz="0 0 0" rpy="0 0 0" />
-        <inertia ixx="0.000000017" ixy="0.0" ixz="0.0" iyy="0.000000017" iyz="0.0" izz="0.000000017"/>
-    </inertial>
-    <visual>
-        <origin xyz="0 0 0" rpy="0 0 0" />
-        <geometry>
-            <mesh filename="package://description_dual/meshes/max_sonar_ez4.dae"/>
-        </geometry>
-    </visual>
-    <collision>
-        <origin xyz="0 0 0" rpy="0 0 0" />
-        <geometry>
-            <box size="0.01 0.01 0.01" />
-        </geometry>
-    </collision>
-</link>
-<joint name="sonar_left_sensor_joint" type="fixed">
-    <parent link="base_link"/>
-    <child link="base_sonar_left"/>
-    <origin xyz="0 0.3 0.09" rpy="0 0 1.57079632679"/>
-</joint>
-<!-- Right sonar sensor -->
-<link name="base_sonar_right">
-    <inertial>
-        <mass value="0.001" />
-        <origin xyz="0 0 0" rpy="0 0 0" />
-        <inertia ixx="0.000000017" ixy="0.0" ixz="0.0" iyy="0.000000017" iyz="0.0" izz="0.000000017"/>
-    </inertial>
-    <visual>
-        <origin xyz="0 0 0" rpy="0 0 0" />
-        <geometry>
-            <mesh filename="package://description_dual/meshes/max_sonar_ez4.dae"/>
-        </geometry>
-    </visual>
-    <collision>
-        <origin xyz="0 0 0" rpy="0 0 0" />
-        <geometry>
-            <box size="0.01 0.01 0.01" />
-        </geometry>
-    </collision>
-</link>
-<joint name="sonar_right_sensor_joint" type="fixed">
-    <parent link="base_link"/>
-    <child link="base_sonar_right"/>
-    <origin xyz="0 -0.3 0.09" rpy="0 0 -1.57079632679"/>
-</joint>
-<!-- Kinect sensor -->
-<link name="base_kinect">
-    <inertial>
-        <mass value="0.01" />
-        <origin xyz="0 0 0" />
-        <inertia ixx="0.001" ixy="0.0" ixz="0.0" iyy="0.001" iyz="0.0" izz="0.001" />
-    </inertial>
-    <visual>
-        <origin xyz="0.0 0.0 0.0" rpy="0 0 0" />
-        <geometry>
-            <mesh filename="package://description_dual/meshes/kinect.dae"/>
-        </geometry>
-    </visual>
-    <collision>
-        <origin xyz="0.0 0.0 0.0" rpy="0 0 0" />
-        <geometry>
-            <mesh filename="package://description_dual/meshes/kinect.dae"/>
-        </geometry>
-    </collision>
-</link>
-<joint name="kinect_camera_joint" type="fixed">
-    <parent link="base_link" />
-    <child link="base_kinect" />
-    <origin xyz="0.41 0 0.465" rpy="0 0 0"/>
-</joint>
-<!-- 1 -->
-<link name="kinect_depth_frame">
-    <inertial>
-        <mass value="0.01" />
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
Commit message: pkg name revised

File: dualarm_mobile_description/urdf/real_robot.urdf.xacro (robot description, xacro)
@@ -44,5 +44,5 @@
             <origin xyz="0 0 0" rpy="0 0 0" />
             <geometry>
-                <mesh filename="package://description_dual/meshes/base_link.STL" />
+                <mesh filename="package://dualarm_mobile_description/meshes/base_link.STL" />
             </geometry>
             <material name="light_grey"/>
@@ -51,5 +51,5 @@
         <origin xyz="0 0 0" rpy="0 0 0" />
             <geometry>
-                <mesh filename="package://description_dual/meshes/base_link.STL" />
+                <mesh filename="package://dualarm_mobile_description/meshes/base_link.STL" />
             </geometry>
         </collision>
@@ -70,5 +70,5 @@
             <origin xyz="0 0 0" rpy="0 0 0" />
             <geometry>
-                <mesh filename="package://description_dual/meshes/br_wheel_link.STL" />
+                <mesh filename="package://dualarm_mobile_description/meshes/br_wheel_link.STL" />
             </geometry>
             <material name="orange"/>
@@ -97,5 +97,5 @@
             <origin xyz="0 0 0" rpy="0 0 0" />
             <geometry>
-                <mesh filename="package://description_dual/meshes/bl_wheel_link.STL" />
+                <mesh filename="package://dualarm_mobile_description/meshes/bl_wheel_link.STL" />
             </geometry>
             <material name="orange"/>
@@ -124,5 +124,5 @@
             <origin xyz="0 0 0" rpy="0 0 0" />
             <geometry>
-                <mesh filename="package://description_dual/meshes/fr_wheel_link.STL" />
+                <mesh filename="package://dualarm_mobile_description/meshes/fr_wheel_link.STL" />
             </geometry>
             <material name="orange"/>
@@ -151,5 +151,5 @@
             <origin xyz="0 0 0" rpy="0 0 0" />
             <geometry>
-                <mesh filename="package://description_dual/meshes/fl_wheel_link.STL" />
+                <mesh filename="package://dualarm_mobile_description/meshes/fl_wheel_link.STL" />
             </geometry>
             <material name="orange"/>
@@ -185,5 +185,5 @@
             <origin xyz="0 0 0.0" rpy="0 0 0"/>
             <geometry>
-                <mesh filename="package://description_dual/meshes/hokuyo.dae" />
+                <mesh filename="package://dualarm_mobile_description/meshes/hokuyo.dae" />
             </geometry>
             <material name="dark_grey"/>
@@ -192,5 +192,5 @@
             <origin xyz="0 0 0.0" rpy="0 0 0"/>
             <geometry>
-                <mesh filename="package://description_dual/meshes/hokuyo_convex.dae" />
+                <mesh filename="package://dualarm_mobile_description/meshes/hokuyo_convex.dae" />
             </geometry>
         </collision>
@@ -211,5 +211,5 @@
             <origin xyz="0 0 0" rpy="0 0 0" />
             <geometry>
-                <mesh filename="package://description_dual/meshes/max_sonar_ez4.dae"/>
+                <mesh filename="package://dualarm_mobile_description/meshes/max_sonar_ez4.dae"/>
             </geometry>
         </visual>
@@ -236,5 +236,5 @@
             <origin xyz="0 0 0" rpy="0 0 0" />
             <geometry>
-                <mesh filename="package://description_dual/meshes/max_sonar_ez4.dae"/>
+                <mesh filename="package://dualarm_mobile_description/meshes/max_sonar_ez4.dae"/>
             </geometry>
         </visual>
@@ -261,5 +261,5 @@
             <origin xyz="0 0 0" rpy="0 0 0" />
             <geometry>
-                <mesh filename="package://description_dual/meshes/max_sonar_ez4.dae"/>
+                <mesh filename="package://dualarm_mobile_description/meshes/max_sonar_ez4.dae"/>
             </geometry>
         </visual>
@@ -286,5 +286,5 @@
             <origin xyz="0 0 0" rpy="0 0 0" />
             <geometry>
-                <mesh filename="package://description_dual/meshes/max_sonar_ez4.dae"/>
+                <mesh filename="package://dualarm_mobile_description/meshes/max_sonar_ez4.dae"/>
             </geometry>
         </visual>
@@ -311,5 +311,5 @@
             <origin xyz="0.0 0.0 0.0" rpy="0 0 0" />
             <geometry>
-                <mesh filename="package://description_dual/meshes/kinect.dae"/>
+                <mesh filename="package://dualarm_mobile_description/meshes/kinect.dae"/>
             </geometry>
         </visual>
@@ -317,5 +317,5 @@
             <origin xyz="0.0 0.0 0.0" rpy="0 0 0" />
             <geometry>
-                <mesh filename="package://description_dual/meshes/kinect.dae"/>
+                <mesh filename="package://dualarm_mobile_description/meshes/kinect.dae"/>
             </geometry>
         </collision>
