Commit message: change some files to fit 2020final robot setup

File: dualarm_mobile_description/urdf/mobile_robot_description_v2.urdf (robot description, URDF)
Before this commit: robot mobile_robot_description_v2, 11 links, 10 joints
Links:
- added link base_footprint
- added link rplidar_front, mass 1e-5; collision mesh filename=package://dualarm_mobile_description/meshes/rplidar.dae scale=0.001 0.001 0.001; visual mesh filename=package://dualarm_mobile_description/meshes/rplidar.dae scale=0.001 0.001 0.001
- added link rplidar_rear, mass 1e-5; collision mesh filename=package://dualarm_mobile_description/meshes/rplidar.dae scale=0.001 0.001 0.001; visual mesh filename=package://dualarm_mobile_description/meshes/rplidar.dae scale=0.001 0.001 0.001
Joints:
- added joint base_joint: type fixed, parent base_footprint, child base_link, origin xyz=0 0 0.117 rpy=0 0 0
- added joint rplidar_front_joint: type fixed, parent base_link, child rplidar_front, origin xyz=0.284 0.189 0.633 rpy=0 0 0, axis 0 1 0
- added joint rplidar_rear_joint: type fixed, parent base_link, child rplidar_rear, origin xyz=-0.284 -0.189 0.633 rpy=0 0 -3.1415926535, axis 0 1 0

Commit message: fix bug

File: dualarm_mobile_description/urdf/mobile_robot_description_v2.urdf (robot description, URDF)
Before this commit: robot mobile_robot_description_v2, 14 links, 13 joints
Joints:
- joint rplidar_front_joint: origin xyz=0.284 0.189 0.633 rpy=0 0 0 -> xyz=0.284 0.189 0.633 rpy=0 0 3.1415926535
- joint rplidar_rear_joint: origin xyz=-0.284 -0.189 0.633 rpy=0 0 -3.1415926535 -> xyz=-0.284 -0.189 0.633 rpy=0 0 0
